File: Beacon/Beacon.kicad_sch (KiCad schematic)
At the start: 0 parts

Commit message: Added MCUs and pheriperal circuits
Other:
- added sheet MCU (MCU_sch.kicad_sch)
Changed lines of the file:
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@@
 	(generator_version "10.0")
 	(paper "A4")
+	(sheet
+		(at 50.8 64.135)
+		(size 30.48 14.605)
+		(exclude_from_sim no)
+		(in_bom yes)
+		(on_board yes)
+		(dnp no)
+		(fields_autoplaced yes)
+		(stroke
+			(width 0.1524)
+			(type solid)
+		)
+		(fill
+			(color 0 0 0 0)
+		)
+		(property "Sheetname" "MCU"
+			(at 50.8 63.4234 0)
+			(show_name no)
+			(do_not_autoplace no)
+			(effects
+				(font
+					(size 1.27 1.27)
+				)
+				(justify left bottom)
+			)
+		)
+		(property "Sheetfile" "MCU_sch.kicad_sch"
+			(at 50.8 79.3246 0)
+			(show_name no)
+			(do_not_autoplace no)
+			(effects
+				(font
+					(size 1.27 1.27)
+				)
+				(justify left top)
+			)
+		)
+		(instances
+			(project "Beacon"
+				(path "/819ea20c-ba44-4e9d-9cd4-06402e06a517"
+					(page "2")
+				)
+			)
+		)
+	)
 	(sheet_instances
 		(path "/"
