File: Beacon/MCU_sch.kicad_sch (KiCad schematic)
At the start: 25 parts, among them J1 Conn_ARM_JTAG_SWD_10, SW1 SW_Push, SW2 SW_Push, U1 STM32U575RITxQ, Y1 16MHz, Y2 32.768KHz

Commit message: minor changes to page info
Parts:
- removed C14, C15: 6p, Capacitor_SMD:C_0805_2012Metric, symbol Device:C
- removed Y2: 32.768KHz, Crystal:Crystal_SMD_3225-4Pin_3.2x2.5mm, symbol Device:Crystal_GND24
- added MT2: Screw_Terminal, TerminalBlock_Phoenix:TerminalBlock_Phoenix_MKDS-1,5-2-5.08_1x02_P5.08mm_Horizontal, symbol Connector:Screw_Terminal_01x02
Connections:
- net +3V3: now also MT2.1 (Pin_1)
- net GND: now also MT2.2 (Pin_2)
- net LSE_IN: no longer names the net of U1.3 (PC14)
- net LSE_OUT: no longer names the net of U1.4 (PC15)
Other:
- note added: "3.3V Line from Beacon"
- note added: "From Main"
- note removed: "32.768KHz Crystal Oscillator"
- company: (none) -> Team Anant - Guru Tanish
- title: (none) -> Beacon Board
